File: Eagle/MainBoard/v3.0/linearSensor.sch (EAGLE design)
At the start: 15 parts, among them X1 FH12-08S-1SH

Commit message: New spectrophotometer board
Parts:
- removed C1: 100pF, rcl:C-EUC0805
- removed LED1, LED5: WHITE, led:LEDCHIP-LED0805
- removed PAD1, PAD2: (no value), wirepad:SMD5
- removed RL1, RL7: 1M, rcl:R-EU_R0805
- removed RL2, RL4: 150, rcl:R-EU_R0805
- removed RL3, RL5, RL6: 100, rcl:R-EU_R0805
- removed U$1: RGB-COMMON-CATHODE, lpatiny:RGB-COMMON-CATHODE
- added C10: 10uF, rcl:R-EU_M0805
- added C11, C3: 100nF, rcl:C-EUC0805K
- added C12: 100nF, rcl:R-EU_M0805
- added C4: 100nF, rcl:C-EUC0805
- added C7: 10uF, rcl:C-EUC0805
- added C8: 22pF, rcl:C-EUC0805K
- added CON1: SPI, lpatiny:TINYISPT
- added D2, D4: 1N581, lpatiny:1N581D1206
- added R13: 1M, rcl:R-EU_M0805
- added R15, R3: 10k, resistor:R-EU_M0805
- added R24, R31: 22, rcl:R-EU_M0805
- added U$2: TSL1402R, lpatiny:TSL1402R
- added U$4: 32U4, adafruit:ATMEGA32U4-AU
- added X3: 16MHz, lpatiny:XTALNX6035
- added X4: MINI-USB, con-cypressindustries:MINI-USB-SCHIELD-32005-201
- C2: value 100pF -> 22pF; device rcl:C-EUC0805 -> rcl:C-EUC0805K
Connections:
- removed net BLUE: RL2.2, X1-4.1
- removed net GREEN: RL3.2, X1-3.1
- removed net N$1: RL4.2, U$1.CGREEN
- removed net N$2: RL3.1, U$1.CBLUE
- removed net N$3: RL2.1, U$1.CRED
- removed net N$4: LED5.A, RL5.1
- removed net N$5: LED1.A, RL6.1
- removed net PULSE: RL1.1, RL7.1, X1-6.1
- removed net RED: RL4.1, X1-2.1
- removed net SENS1: C2.1, PAD1.P, RL7.2, X1-7.1
- removed net SENS2: C1.1, PAD2.P, RL1.2, X1-8.1
- removed net WHITE: RL5.2, RL6.2, X1-5.1
- new net +5V/1: C10.2, C12.2, C4.2, D2.C, D4.C, R15.2, U$2.VDD, U$4.AVCC, U$4.AVCC1, U$4.UVCC, U$4.VCC, U$4.VCC1
- new net A0: U$4.PF7(ADC7(TDI)
- new net A1: U$2.AO1, U$4.PF6(ADC6/TDO)
- new net A2: U$2.AO2, U$4.PF5(ADC5/TMS)
- new net A3: U$4.PF4(ADC4/TCK), X1-2.1
- new net A4: U$4.PF1(ADC1), X1-1.1
- new net A5: U$4.PF0(ADC0)
- new net AREF: C11.1, U$4.AREF
- new net CS: U$4.PD4(ICP1/ADC8)
- new net D+USB: R24.2, X4G$1.3
- new net D-USB: R31.2, X4G$1.2
- new net D10*: U$4.PB6(OC1B/OC4B/ADC13)
- new net D11*: U$4.PB7(OC0A/OC1C/RTS), X1-7.1
- new net D12*: U$4.PD6(T1/ADC9/!OC4D)
- new net D13*: U$4.PC7(ICP3/CLK0/OC4A), X1-5.1
- new net D5*: U$4.PC6(OC3A/!OC4A), X1-3.1
- new net D6*: U$4.PD7(OC4D/ADC10/T0), X1-6.1
- new net D7*: U$2.SI1, U$2.SI2, U$4.PE6(INT.6/AIN0)
- new net D8*: U$2.CLK, U$4.PB4(ADC11)
- new net D9*: U$4.PB5(OC1A/ADC12/!OC4B), X1-4.1
- new net HWB: R3.2, U$4.PE2(!HWB)
- new net ISP+5V: CON1.VCC, D2.A
- new net MISO: CON1.MISO, U$4.PB3(PDO/MISO)
- new net MOSI: CON1.MOSI, U$4.PB2(PDI/MOSI)
- new net N$16: C3.2, U$4.UCAP
- new net N$42: C8.2, R13.2, U$4.XTAL1, X3.P$2
- new net RD+: R24.1, U$4.D+
- new net RD-: R31.1, U$4.D-
- new net RESET: CON1.RESET, R15.1, U$4./RESET
- new net RX: U$4.PD2(INT2/RXD1)
- new net RXLED: U$4.PB0(SS)
- new net SCK: CON1.SCK, U$4.PB1(SCK)
- new net SCL: U$4.PD0(INT0/OC0B/SCL)
- new net SDA: U$4.PD1(INT1/SDA)
- new net TX: U$4.PD3(INT3/TXD1)
- new net TXLED: U$4.PD5(XCK/CTS)
- new net VUSB: C7.2, D4.A, U$4.VBUS, X4G$1.1
- new net XTAL1: C2.2, R13.1, U$4.XTAL2, X3.P$1
- net GND: now also C10.1, C11.2, C12.1, C2.1, C3.1, C4.1, C7.1, C8.1, CON1.GND, R3.1, U$2.GND1, U$2.GND2, U$4.GND, U$4.GND1, U$4.GND2, U$4.GND3, U$4.UGND, X1-8.1, X4G$1.5; no longer C1.2, C2.2, LED1.C, LED5.C, U$1.A2, X1-1.1
Other:
- note added: "ATMega32u4"
- note added: "BLUE"
- note added: "GND"
- note added: "GREEN"
- note added: "PULSE"
- note added: "RED"
- note added: "SENS1"
- note added: "SENS2"
- note added: "WHITE"
- moved on the sheet: C2, X1-1, X1-2, X1-3, X1-4, X1-5, X1-6, X1-7, X1-8
